File: Hardware/KiCad_Stator/KiCad_Stator.kicad_sch (KiCad schematic)
At the start: 0 parts

Commit message: feat:prototype v0.1
Parts:
- added A1: A, Connector_PinHeader_1.27mm:PinHeader_1x01_P1.27mm_Vertical, symbol Connector:Conn_01x01_Pin
- added B1: B, Connector_PinHeader_1.27mm:PinHeader_1x01_P1.27mm_Vertical, symbol Connector:Conn_01x01_Pin
- added C1: C, Connector_PinHeader_1.27mm:PinHeader_1x01_P1.27mm_Vertical, symbol Connector:Conn_01x01_Pin
- added H1: MountingHole, MountingHole:MountingHole_5.3mm_M5, symbol Mechanical:MountingHole
- added NT1, NT2, NT3: NetTie_2, NetTie:NetTie-2_SMD_Pad0.5mm, symbol Device:NetTie_2
Connections:
- new net A: A1.1 (Pin_1), NT1.2
- new net B: B1.1 (Pin_1), NT2.2
- new net C: C1.1 (Pin_1), NT3.2
- new net GND: NT1.1, NT2.1, NT3.1
