File: Hardware/KiCad_FOC-ESC/FET_Driver.kicad_sch (KiCad schematic)
At the start: 1 part, among them IC1 DRV8300DPWR

Commit message: inited Software (#7)
Parts:
- IC1: footprint SOP65P640X120-20N -> SamacSys_Parts:SOP65P640X120-20N
Changed lines of the file:
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@@
 			)
 		)
-		(property "Footprint" "SOP65P640X120-20N"
+		(property "Footprint" "SamacSys_Parts:SOP65P640X120-20N"
 			(at 91.44 168.58 0)
 			(hide yes)
