File: Hardware/KiCad_FOC-ESC/FETs.kicad_sch (KiCad schematic)
At the start: 6 parts, among them Q1 NTTFS5D6N08XLTAG, Q2 NTTFS5D6N08XLTAG, Q3 NTTFS5D6N08XLTAG, Q4 NTTFS5D6N08XLTAG, Q5 NTTFS5D6N08XLTAG, Q6 NTTFS5D6N08XLTAG

Commit message: inited Software (#7)
Parts:
- Q1, Q2, Q3, Q4, Q5, Q6: footprint NVTFS007N08HLTAG -> SamacSys_Parts:NVTFS007N08HLTAG
Changed lines of the file:
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@@
 			)
 		)
-		(property "Footprint" "NVTFS007N08HLTAG"
+		(property "Footprint" "SamacSys_Parts:NVTFS007N08HLTAG"
 			(at 118.11 183.82 0)
 			(hide yes)
@@
 			)
 		)
-		(property "Footprint" "NVTFS007N08HLTAG"
+		(property "Footprint" "SamacSys_Parts:NVTFS007N08HLTAG"
 			(at 148.59 159.69 0)
 			(hide yes)
@@
 			)
 		)
-		(property "Footprint" "NVTFS007N08HLTAG"
+		(property "Footprint" "SamacSys_Parts:NVTFS007N08HLTAG"
 			(at 148.59 183.82 0)
 			(hide yes)
@@
 			)
 		)
-		(property "Footprint" "NVTFS007N08HLTAG"
+		(property "Footprint" "SamacSys_Parts:NVTFS007N08HLTAG"
 			(at 118.11 159.69 0)
 			(hide yes)
@@
 			)
 		)
-		(property "Footprint" "NVTFS007N08HLTAG"
+		(property "Footprint" "SamacSys_Parts:NVTFS007N08HLTAG"
 			(at 118.11 209.22 0)
 			(hide yes)
@@
 			)
 		)
-		(property "Footprint" "NVTFS007N08HLTAG"
+		(property "Footprint" "SamacSys_Parts:NVTFS007N08HLTAG"
 			(at 148.59 209.22 0)
 			(hide yes)
