File: Hardware/KiCad_FOC-ESC/FETs.kicad_sch (KiCad schematic)
At the start: 0 parts

Commit message: initial connections
Parts:
- added C18: 1uF, Capacitor_SMD:C_0603_1608Metric, symbol Device:C
- added C21, C22, C23: 100nF, Capacitor_SMD:C_0402_1005Metric, symbol Device:C
- added IC1: DRV8300DPWR, SamacSys_Parts:SOP65P640X120-20N, symbol SamacSys_Parts:DRV8300DPWR
Connections:
- net GHA: now also IC1.19 (GHA)
- net GHB: now also IC1.16 (GHB)
- net GHC: now also IC1.13 (GHC)
- net GLA: now also IC1.11 (GLA)
- net GLB: now also IC1.10 (GLB)
- net GLC: now also IC1.9 (GLC)
- net GND: now also C18.1, IC1.8 (GND)
- new net: C18.2, IC1.7 (GVDD)
- new net BSTA: C21.2, IC1.20 (BSTA)
- new net BSTB: C22.2, IC1.17 (BSTB)
- new net BSTC: C23.2, IC1.14 (BSTC)
- new net INHA: IC1.1 (INHA)
- new net INHB: IC1.2 (INHB)
- new net INHC: IC1.3 (INHC)
- new net INLA: IC1.4 (INLA)
- new net INLB: IC1.5 (INLB)
- new net INLC: IC1.6 (INLC)
- new net SHA: C21.1, IC1.18 (SHA)
- new net SHB: C22.1, IC1.15 (SHB)
- new net SHC: C23.1, IC1.12 (SHC)
Other:
- sheet HalfBridgeA ports: added SH; removed none
- sheet HalfBridgeB ports: added SH; removed none
- sheet HalfBridgeC ports: added SH; removed none
