File: Hardware/KiCad_FOC-ESC/FETs.kicad_sch (KiCad schematic)
At the start: 5 parts, among them IC1 DRV8300DPWR

Commit message: changed formfactor, driver, output stage (#14)
Co-authored-by: CTTOSP <255604560+CTTOSP@users.noreply.github.com>
Parts:
- removed C18: 1uF, Capacitor_SMD:C_0603_1608Metric, symbol Device:C
- removed C21, C22, C23: 100nF, Capacitor_SMD:C_0402_1005Metric, symbol Device:C
- removed IC1: DRV8300DPWR, SamacSys_Parts:SOP65P640X120-20N, symbol SamacSys_Parts:DRV8300DPWR
- added NT1, NT2, NT3: NetTie_2, NetTie:NetTie-2_SMD_Pad0.5mm, symbol Device:NetTie_2
Connections:
- new net DRV8320S_1/SPA: NT1.1
- new net DRV8320S_1/SPB: NT2.1
- new net DRV8320S_1/SPC: NT3.1
- new net SLA: NT1.2
- new net SLB: NT2.2
- new net SLC: NT3.2
Other:
- added sheet DRV8320S_1 (DRV8320S.kicad_sch)
- sheet HalfBridgeA ports: added SL; removed none
- sheet HalfBridgeB ports: added SL; removed none
- sheet HalfBridgeC ports: added SL; removed none
