File: Hardware/KiCad_FOC-ESC/angle_sens.kicad_sch (KiCad schematic)
At the start: 1 part, among them IC6 MA702GQ-P

Commit message: inited Software (#7)
Parts:
- IC6: footprint QFN50P300X300X100-17N-D -> SamacSys_Parts:QFN50P300X300X100-17N-D
Changed lines of the file:
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@@
 			)
 		)
-		(property "Footprint" "QFN50P300X300X100-17N-D"
+		(property "Footprint" "SamacSys_Parts:QFN50P300X300X100-17N-D"
 			(at 140.97 171.12 0)
 			(hide yes)

Commit message: ready
Parts:
- added U3: MT6701CT, Package_SO:SO-8_3.9x4.9mm_P1.27mm, symbol Sensor_Magnetic:MT6701CT
Changed lines of the file:
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@@
 	(paper "A4")
+	(symbol
+		(lib_id "Sensor_Magnetic:MT6701CT")
+		(at 46.99 90.17 0)
+		(unit 1)
+		(body_style 1)
+		(exclude_from_sim no)
+		(in_bom yes)
+		(on_board yes)
+		(in_pos_files yes)
+		(dnp no)
+		(fields_autoplaced yes)
+		(property "Reference" "U3"
+			(at 49.1333 69.85 0)
+			(show_name no)
+			(do_not_autoplace no)
+			(effects
+				(font
+					(size 1.27 1.27)
+				)
+				(justify left)
+			)
+		)
+		(property "Value" "MT6701CT"
+			(at 49.1333 72.39 0)
+			(show_name no)
+			(do_not_autoplace no)
+			(effects
+				(font
+					(size 1.27 1.27)
+				)
+				(justify left)
+			)
+		)
+		(property "Footprint" "Package_SO:SO-8_3.9x4.9mm_P1.27mm"
+			(at 46.99 120.65 0)
+			(hide yes)
+			(show_name no)
+			(do_not_autoplace no)
+			(effects
+				(font
+					(size 1.27 1.27)
+				)
+			)
+		)
+		(property "Datasheet" "https://www.magntek.com.cn/upload/MT6701_Rev.1.5.pdf"
+			(at 46.99 123.19 0)
+			(hide yes)
+			(show_name no)
+			(do_not_autoplace no)
+			(effects
+				(font
+					(size 1.27 1.27)
+				)
+			)
+		)
+		(property "Description" "Hall Based Angle Position Encoder Sensor, I2C, SSI, ABZ & UVW interfaces, 3.3..5V supply, SOIC-8"
+			(at 46.99 90.17 0)
+			(hide yes)
+			(show_name no)
+			(do_not_autoplace no)
+			(effects
+				(font
+					(size 1.27 1.27)
+				)
+			)
+		)
+		(pin "5"
+		)
+		(pin "3"
+		)
+		(pin "1"
+		)
+		(pin "2"
+		)
+		(pin "4"
+		)
+		(pin "6"
+		)
+		(pin "8"
+		)
+		(pin "7"
+		)
+		(instances
+			(project "KiCad_FOC-ESC"
+				(path "/5aa129d7-7a76-48d9-8008-691cf751c140/3fb604c9-4375-4b1d-95f1-f4834b76ca89"
+					(reference "U3")
+					(unit 1)
+				)
+			)
+		)
+	)
 	(symbol
 		(lib_id "SamacSys_Parts:MA702GQ-P")
