File: Hardware/KiCad_FOC-ESC/current_sens.kicad_sch (KiCad schematic)
At the start: 3 parts, among them IC2 TSC1801BILT, IC3 TSC1801BILT, IC4 TSC1801BILT

Commit message: inited Software (#7)
Parts:
- IC2, IC3, IC4: footprint SOT95P280X145-6N -> SamacSys_Parts:SOT95P280X145-6N
Changed lines of the file:
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@@
 			)
 		)
-		(property "Footprint" "SOT95P280X145-6N"
+		(property "Footprint" "SamacSys_Parts:SOT95P280X145-6N"
 			(at 113.03 169.85 0)
 			(hide yes)
@@
 			)
 		)
-		(property "Footprint" "SOT95P280X145-6N"
+		(property "Footprint" "SamacSys_Parts:SOT95P280X145-6N"
 			(at 113.03 186.36 0)
 			(hide yes)
@@
 			)
 		)
-		(property "Footprint" "SOT95P280X145-6N"
+		(property "Footprint" "SamacSys_Parts:SOT95P280X145-6N"
 			(at 113.03 152.07 0)
 			(hide yes)

Commit message: ready
Parts:
- added R1, R2, R3: PMR100HZP7FV1L00, PMR100HZP7FV1L00, symbol SamacSys_Parts:PMR100HZP7FV1L00
