File: Hardware/KiCad_FOC-ESC/CMOS_Oscillator.kicad_sch (KiCad schematic)
At the start: 2 parts, among them Y1 ASDDV-16.000MHZ-LR-T

Commit message: initial connections
Connections:
- net +3.3V renamed +3V3
Changed lines of the file:
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@@
 	)
 	(symbol
-		(lib_id "power:+3.3V")
+		(lib_id "power:+3V3")
 		(at 80.01 68.58 0)
 		(unit 1)
@@
 		(in_pos_files yes)
 		(dnp no)
-		(property "Reference" "#PWR0105"
+		(fields_autoplaced yes)
+		(property "Reference" "#PWR051"
 			(at 80.01 72.39 0)
 			(hide yes)
@@
 			)
 		)
-		(property "Value" "+3.3V"
-			(at 80.01 63.246 0)
+		(property "Value" "+3V3"
+			(at 80.01 63.5 0)
 			(show_name no)
 			(do_not_autoplace no)
@@
 			)
 		)
-		(property "Description" "Power symbol creates a global label with name \"+3.3V\""
+		(property "Description" "Power symbol creates a global label with name \"+3V3\""
 			(at 80.01 68.58 0)
 			(hide yes)
@@
 			(project "KiCad_FOC-ESC"
 				(path "/5aa129d7-7a76-48d9-8008-691cf751c140/dd72814a-2d5c-4d6c-a81f-25fb4510d80e"
-					(reference "#PWR0105")
+					(reference "#PWR051")
 					(unit 1)
 				)
@@
 	)
 	(symbol
-		(lib_id "power:+3.3V")
+		(lib_id "power:GND")
+		(at 80.01 88.9 0)
+		(unit 1)
+		(body_style 1)
+		(exclude_from_sim no)
+		(in_bom yes)
+		(on_board yes)
+		(in_pos_files yes)
+		(dnp no)
+		(property "Reference" "#PWR0106"
+			(at 80.01 95.25 0)
+			(hide yes)
+			(show_name no)
+			(do_not_autoplace no)
+			(effects
+				(font
+					(size 1.27 1.27)
+				)
+			)
+		)
+		(property "Value" "GND"
+			(at 80.01 92.964 0)
+			(show_name no)
+			(do_not_autoplace no)
+			(effects
+				(font
+					(size 1.27 1.27)
+				)
+			)
+		)
+		(property "Footprint" ""
+			(at 80.01 88.9 0)
+			(hide yes)
+			(show_name no)
+			(do_not_autoplace no)
+			(effects
+				(font
+					(size 1.27 1.27)
+				)
+			)
+		)
+		(property "Datasheet" ""
+			(at 80.01 88.9 0)
+			(hide yes)
+			(show_name no)
+			(do_not_autoplace no)
+			(effects
+				(font
+					(size 1.27 1.27)
+				)
+			)
+		)
+		(property "Description" "Power symbol creates a global label with name \"GND\" , ground"
+			(at 80.01 88.9 0)
+			(hide yes)
+			(show_name no)
+			(do_not_autoplace no)
+			(effects
+				(font
+					(size 1.27 1.27)
+				)
+			)
+		)
+		(pin "1"
+		)
+		(instances
+			(project "KiCad_FOC-ESC"
+				(path "/5aa129d7-7a76-48d9-8008-691cf751c140/dd72814a-2d5c-4d6c-a81f-25fb4510d80e"
+					(reference "#PWR0106")
+					(unit 1)
+				)
+			)
+		)
+	)
+	(symbol
+		(lib_id "power:+3V3")
 		(at 86.36 68.58 0)
 		(unit 1)
@@
 		(in_pos_files yes)
 		(dnp no)
-		(property "Reference" "#PWR0109"
+		(fields_autoplaced yes)
+		(property "Reference" "#PWR050"
 			(at 86.36 72.39 0)
 			(hide yes)
@@
 			)
 		)
-		(property "Value" "+3.3V"
-			(at 86.36 63.246 0)
+		(property "Value" "+3V3"
+			(at 86.36 63.5 0)
 			(show_name no)
 			(do_not_autoplace no)
@@
 			)
 		)
-		(property "Description" "Power symbol creates a global label with name \"+3.3V\""
+		(property "Description" "Power symbol creates a global label with name \"+3V3\""
 			(at 86.36 68.58 0)
 			(hide yes)
@@
 			(project "KiCad_FOC-ESC"
 				(path "/5aa129d7-7a76-48d9-8008-691cf751c140/dd72814a-2d5c-4d6c-a81f-25fb4510d80e"
-					(reference "#PWR0109")
-					(unit 1)
-				)
-			)
-		)
-	)
-	(symbol
-		(lib_id "power:GND")
-		(at 80.01 88.9 0)
-		(unit 1)
-		(body_style 1)
-		(exclude_from_sim no)
-		(in_bom yes)
-		(on_board yes)
-		(in_pos_files yes)
-		(dnp no)
-		(property "Reference" "#PWR0106"
-			(at 80.01 95.25 0)
-			(hide yes)
-			(show_name no)
-			(do_not_autoplace no)
-			(effects
-				(font
-					(size 1.27 1.27)
-				)
-			)
-		)
-		(property "Value" "GND"
-			(at 80.01 92.964 0)
-			(show_name no)
-			(do_not_autoplace no)
-			(effects
-				(font
-					(size 1.27 1.27)
-				)
-			)
-		)
-		(property "Footprint" ""
-			(at 80.01 88.9 0)
-			(hide yes)
-			(show_name no)
-			(do_not_autoplace no)
-			(effects
-				(font
-					(size 1.27 1.27)
-				)
-			)
-		)
-		(property "Datasheet" ""
-			(at 80.01 88.9 0)
-			(hide yes)
-			(show_name no)
-			(do_not_autoplace no)
-			(effects
-				(font
-					(size 1.27 1.27)
-				)
-			)
-		)
-		(property "Description" "Power symbol creates a global label with name \"GND\" , ground"
-			(at 80.01 88.9 0)
-			(hide yes)
-			(show_name no)
-			(do_not_autoplace no)
-			(effects
-				(font
-					(size 1.27 1.27)
-				)
-			)
-		)
-		(pin "1"
-		)
-		(instances
-			(project "KiCad_FOC-ESC"
-				(path "/5aa129d7-7a76-48d9-8008-691cf751c140/dd72814a-2d5c-4d6c-a81f-25fb4510d80e"
-					(reference "#PWR0106")
-					(unit 1)
-				)
+					(reference "#PWR050")
+					(unit 1)
+				)
