File: Hardware/KiCad_FOC-ESC/HalfBridge.kicad_sch (KiCad schematic)
At the start: 6 parts, among them IC2 TSC1801BILT, J1 Conn_01x01_Socket, Q1 NTTFS5D6N08XLTAG, Q2 NTTFS5D6N08XLTAG

Commit message: initial connections
Parts:
- removed J1: Conn_01x01_Socket, Connector_PinHeader_2.54mm:PinHeader_1x01_P2.54mm_Vertical, symbol Connector:Conn_01x01_Socket
- added C14: 100nF, Capacitor_SMD:C_0402_1005Metric, symbol Device:C
Connections:
- net GND: now also C14.2
- net MP renamed SH
- net Vref renamed +1V5
- net +1V5: now also C14.1
