File: Hardware/KiCad_FOC-ESC/HalfBridge.kicad_sch (KiCad schematic)
At the start: 6 parts, among them IC2 TSC1801BILT, Q1 NTTFS5D6N08XLTAG, Q2 NTTFS5D6N08XLTAG

Commit message: changed formfactor, driver, output stage (#14)
Co-authored-by: CTTOSP <255604560+CTTOSP@users.noreply.github.com>
Parts:
- R4: footprint RESC3225X67N -> SamacSys_Parts:RESC3225X67N
Connections:
- net GND1 renamed SL
Changed lines of the file:
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@@
 	(paper "A4")
+	(junction
+		(at 74.93 129.54)
+		(diameter 0)
+		(color 0 0 0 0)
+	)
 	(junction
 		(at 133.35 139.7)
@@
 	(wire
 		(pts
+			(xy 78.74 129.54) (xy 74.93 129.54)
+		)
+		(stroke
+			(width 0)
+			(type default)
+		)
+	)
+	(wire
+		(pts
 			(xy 128.27 100.33) (xy 128.27 93.98)
 		)
@@
 	(wire
 		(pts
+			(xy 74.93 129.54) (xy 74.93 125.73)
+		)
+		(stroke
+			(width 0)
+			(type default)
+		)
+	)
+	(wire
+		(pts
 			(xy 72.39 64.77) (xy 72.39 71.12)
 		)
@@
 	(wire
 		(pts
-			(xy 74.93 132.08) (xy 74.93 125.73)
+			(xy 74.93 132.08) (xy 74.93 129.54)
 		)
 		(stroke
@@
 			)
 			(justify right)
+		)
+	)
+	(hierarchical_label "SL"
+		(shape input)
+		(at 78.74 129.54 0)
+		(effects
+			(font
+				(size 1.27 1.27)
+			)
+			(justify left)
 		)
 	)
@@
 			)
 		)
-		(property "Footprint" "RESC3225X67N"
+		(property "Footprint" "SamacSys_Parts:RESC3225X67N"
 			(at 171.12 135.89 0)
 			(hide yes)

Commit message: edited routs
Parts:
- added NT4: NetTie_2, NetTie:NetTie-2_SMD_Pad0.5mm, symbol Device:NetTie_2
Connections:
- net GND: now also NT4.2; no longer IC2.5 (IN-)
- new net: IC2.5 (IN-), NT4.1
Changed lines of the file:
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@@
+	(wire
+		(pts
+			(xy 128.27 80.01) (xy 128.27 86.36)
+		)
+		(stroke
+			(width 0)
+			(type default)
+		)
+	)
 	(wire
 		(pts
@@
 	(wire
 		(pts
-			(xy 128.27 100.33) (xy 128.27 93.98)
-		)
-		(stroke
-			(width 0)
-			(type default)
-		)
-	)
-	(wire
-		(pts
 			(xy 82.55 114.3) (xy 82.55 107.95)
 		)
@@
 		(pts
 			(xy 125.73 135.89) (xy 128.27 135.89)
+		)
+		(stroke
+			(width 0)
+			(type default)
+		)
+	)
+	(wire
+		(pts
+			(xy 128.27 91.44) (xy 128.27 100.33)
 		)
 		(stroke
@@
 	)
 	(label "GND2"
-		(at 128.27 93.98 270)
+		(at 128.27 80.01 270)
 		(effects
 			(font
@@
 		)
 	)
+	(symbol
+		(lib_id "Device:NetTie_2")
+		(at 128.27 88.9 90)
+		(unit 1)
+		(body_style 1)
+		(exclude_from_sim no)
+		(in_bom no)
+		(on_board yes)
+		(in_pos_files yes)
+		(dnp no)
+		(fields_autoplaced yes)
+		(property "Reference" "NT4"
+			(at 129.54 87.6299 90)
+			(show_name no)
+			(do_not_autoplace no)
+			(effects
+				(font
+					(size 1.27 1.27)
+				)
+				(justify right)
+			)
+		)
+		(property "Value" "NetTie_2"
+			(at 129.54 90.1699 90)
+			(show_name no)
+			(do_not_autoplace no)
+			(effects
+				(font
+					(size 1.27 1.27)
+				)
+				(justify right)
+			)
+		)
+		(property "Footprint" "NetTie:NetTie-2_SMD_Pad0.5mm"
+			(at 128.27 88.9 0)
+			(hide yes)
+			(show_name no)
+			(do_not_autoplace no)
+			(effects
+				(font
+					(size 1.27 1.27)
+				)
+			)
+		)
+		(property "Datasheet" ""
+			(at 128.27 88.9 0)
+			(hide yes)
+			(show_name no)
+			(do_not_autoplace no)
+			(effects
+				(font
+					(size 1.27 1.27)
+				)
+			)
+		)
+		(property "Description" "Net tie, 2 pins"
+			(at 128.27 88.9 0)
+			(hide yes)
+			(show_name no)
+			(do_not_autoplace no)
+			(effects
+				(font
+					(size 1.27 1.27)
+				)
+			)
+		)
+		(pin "1"
+		)
+		(pin "2"
+		)
+		(instances
+			(project "KiCad_FOC-ESC"
+				(path "/5aa129d7-7a76-48d9-8008-691cf751c140/3e4aa878-e28e-4c56-93d1-7a801dda56f4/d6e27ad6-1601-412e-bf7b-bb5db89d9af0"
+					(reference "NT6")
+					(unit 1)
+				)
+				(path "/5aa129d7-7a76-48d9-8008-691cf751c140/3e4aa878-e28e-4c56-93d1-7a801dda56f4/d755ae58-9e58-4fca-bf5c-9be49bc49c40"
+					(reference "NT5")
+					(unit 1)
+				)
+				(path "/5aa129d7-7a76-48d9-8008-691cf751c140/3e4aa878-e28e-4c56-93d1-7a801dda56f4/eb5eeb7a-42d1-404c-b4dc-a9c559d81741"
+					(reference "NT4")
+					(unit 1)
+				)
+			)
+		)
+	)
