File: Hardware/KiCad_FOC-ESC/KiCad_FOC-ESC.kicad_pcb (KiCad board)
At the start: 4 copper layers, 41 x 41 mm, 35 parts, among them IC1 DRV8300DPWR, IC2 TSC1801BILT, IC3 TSC1801BILT, IC4 TSC1801BILT, IC6 MA702GQ-P, J1 Conn_01x01_Socket, J2 Conn_01x01_Socket, J3 Conn_01x01_Socket, Q1 NTTFS5D6N08XLTAG, Q2 NTTFS5D6N08XLTAG, Q3 NTTFS5D6N08XLTAG, Q4 NTTFS5D6N08XLTAG, Q5 NTTFS5D6N08XLTAG, Q6 NTTFS5D6N08XLTAG, U1 STM32G473RCTx, U3 MT6701CT, Y1 ASDDV-16.000MHZ-LR-T

Commit message: initial connections
Parts:
- removed J1, J2, J3: Conn_01x01_Socket, Connector_PinHeader_2.54mm:PinHeader_1x01_P2.54mm_Vertical
- removed LED1: 4684, SamacSys_Parts1:4684
- removed PS1: REF3030AIDBZR, SamacSys_Parts:SOT96P240X105-3N
- added C13: 100nF, Capacitor_SMD:C_0402_1005Metric, F.Cu at (133.3, 102.1)
- added C14: 100nF, Capacitor_SMD:C_0402_1005Metric, F.Cu at (152.6, 100.8)
- added C15: 100nF, Capacitor_SMD:C_0402_1005Metric, F.Cu at (147.5, 105.4)
- added C16: 100nF, Capacitor_SMD:C_0402_1005Metric, F.Cu at (139.9, 104.5)
- added C17: 100nF, Capacitor_SMD:C_0402_1005Metric, F.Cu at (133.1, 98.1)
- added C18: 1uF, Capacitor_SMD:C_0603_1608Metric, F.Cu at (155.3, 89.3)
- added C19: 100nF, Capacitor_SMD:C_0402_1005Metric, F.Cu at (134.7, 99.8)
- added C21: 100nF, Capacitor_SMD:C_0402_1005Metric, F.Cu at (159.4, 100.1)
- added C22: 100nF, Capacitor_SMD:C_0402_1005Metric, F.Cu at (157.4, 100.1)
- added C23: 100nF, Capacitor_SMD:C_0402_1005Metric, F.Cu at (155.5, 99.8)
- added D1: WS2812B-2020, LED_SMD:LED_WS2812B-2020_PLCC4_2.0x2.0mm, F.Cu at (144.0, 80.4)
- added D2: WS2812B-2020, LED_SMD:LED_WS2812B-2020_PLCC4_2.0x2.0mm, F.Cu at (147.1, 80.4)
- added D3: WS2812B-2020, LED_SMD:LED_WS2812B-2020_PLCC4_2.0x2.0mm, F.Cu at (150.2, 80.4)
- added D4: WS2812B-2020, LED_SMD:LED_WS2812B-2020_PLCC4_2.0x2.0mm, F.Cu at (153.4, 80.4)
- added IC5: REF2030AIDDCR, SamacSys_Parts:SOT95P280X110-5N, F.Cu at (131.7, 100.0)
- added U802: ZLDO1117Q, Package_TO_SOT_SMD:SOT-223-3_TabPin2, F.Cu at (148.9, 89.0)
- C7: value 10nF -> 100nF
- moved Q5 81.7 mm to (133.3, 109.9), turned to -45 degrees
- moved Q6 80.5 mm to (130.7, 107.2), turned to 135 degrees
- moved R6 78.4 mm to (134.7, 105.8), turned to 135 degrees
- moved C12 76.5 mm to (136.7, 101.3), turned to -135 degrees
- moved IC4 76.0 mm to (137.7, 103.5), turned to -135 degrees
- moved U1 71.3 mm to (136.2, 88.2)
- moved C11 63.0 mm to (142.9, 105.4), turned to -90 degrees
- moved IC3 61.0 mm to (145.2, 106.2)
- moved Q4 61.0 mm to (142.8, 113.8)
- moved R5 61.0 mm to (144.7, 110.0)
- moved Q3 61.0 mm to (146.6, 113.9)
- moved U3 59.0 mm to (144.5, 96.2)
- moved C7 55.7 mm to (146.0, 82.6), turned to -90 degrees
- moved IC6 53.5 mm to (144.5, 96.2)
- moved C5 52.5 mm to (143.4, 84.6), turned to 90 degrees
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Connections:
- net Vref renamed +1V5
- C103 pad 2: +3.3V -> +3V3
- C2 pad 1: GND -> +3V3
- C2 pad 2: +3V3 -> GND
- C8 pad 2: +3V3 -> +3V
- C9 pad 2: +3V3 -> +3V
- IC1 pad 7: unconnected-(IC1-GVDD-Pad7) -> Net-(IC1-GVDD)
- IC1 pad 8: unconnected-(IC1-GND-Pad8) -> GND
- IC2 pad 6: /FETs/HalfBridgeA/OUT -> OUT1
- IC3 pad 6: /FETs/HalfBridgeB/OUT -> OUT2
- IC4 pad 6: /FETs/HalfBridgeC/OUT -> OUT3
- Q1 pad 1: /FETs/HalfBridgeA/MP -> SHA
- Q1 pad 12: /FETs/HalfBridgeA/MP -> SHA
- Q1 pad 2: /FETs/HalfBridgeA/MP -> SHA
- Q1 pad 3: /FETs/HalfBridgeA/MP -> SHA
- Q2 pad 10: /FETs/HalfBridgeA/MP -> SHA
- Q2 pad 11: /FETs/HalfBridgeA/MP -> SHA
- Q2 pad 5: /FETs/HalfBridgeA/MP -> SHA
- Q2 pad 6: /FETs/HalfBridgeA/MP -> SHA
- Q2 pad 7: /FETs/HalfBridgeA/MP -> SHA
- Q2 pad 8: /FETs/HalfBridgeA/MP -> SHA
- Q2 pad 9: /FETs/HalfBridgeA/MP -> SHA
- Q3 pad 1: /FETs/HalfBridgeB/MP -> SHB
- Q3 pad 12: /FETs/HalfBridgeB/MP -> SHB
- Q3 pad 2: /FETs/HalfBridgeB/MP -> SHB
- Q3 pad 3: /FETs/HalfBridgeB/MP -> SHB
- Q4 pad 10: /FETs/HalfBridgeB/MP -> SHB
- Q4 pad 11: /FETs/HalfBridgeB/MP -> SHB
- Q4 pad 5: /FETs/HalfBridgeB/MP -> SHB
- Q4 pad 6: /FETs/HalfBridgeB/MP -> SHB
- Q4 pad 7: /FETs/HalfBridgeB/MP -> SHB
- Q4 pad 8: /FETs/HalfBridgeB/MP -> SHB
- Q4 pad 9: /FETs/HalfBridgeB/MP -> SHB
- Q5 pad 1: /FETs/HalfBridgeC/MP -> SHC
- Q5 pad 12: /FETs/HalfBridgeC/MP -> SHC
- Q5 pad 2: /FETs/HalfBridgeC/MP -> SHC
- Q5 pad 3: /FETs/HalfBridgeC/MP -> SHC
- Q6 pad 10: /FETs/HalfBridgeC/MP -> SHC
- Q6 pad 11: /FETs/HalfBridgeC/MP -> SHC
- Q6 pad 5: /FETs/HalfBridgeC/MP -> SHC
- Q6 pad 6: /FETs/HalfBridgeC/MP -> SHC
- Q6 pad 7: /FETs/HalfBridgeC/MP -> SHC
- Q6 pad 8: /FETs/HalfBridgeC/MP -> SHC
- Q6 pad 9: /FETs/HalfBridgeC/MP -> SHC
- U1 pad 1: unconnected-(U1-VBAT-Pad1) -> +3V3
- U1 pad 17: unconnected-(U1-PA3-Pad17) -> OUT3
- U1 pad 20: unconnected-(U1-PA6-Pad20) -> OUT2
- U1 pad 25: unconnected-(U1-PB1-Pad25) -> OUT1
- U1 pad 28: +3V3 -> +3V
- U1 pad 35: unconnected-(U1-PB13-Pad35) -> INLC
- U1 pad 36: unconnected-(U1-PB14-Pad36) -> INLB
- U1 pad 42: unconnected-(U1-PA8-Pad42) -> INHA
- U1 pad 43: unconnected-(U1-PA9-Pad43) -> INHB
- U1 pad 44: unconnected-(U1-PA10-Pad44) -> INHC
- U1 pad 45: unconnected-(U1-PA11-Pad45) -> INLA
- Y1 pad 4: +3.3V -> +3V3
Routing:
- net +3V3: track 3.94 -> 129.0 mm, vias 0 -> 15
- net +5V: track 0.00 -> 45.2 mm, vias 0 -> 5
- net +1V5: track 0.00 -> 38.3 mm, vias 0 -> 6
- net SHC: track 0.00 -> 35.9 mm, vias 0 -> 26
- net GHC: track 0.99 -> 32.7 mm, vias 1 -> 2
- net GLC: track 0.00 -> 30.7 mm, vias 0 -> 2
- net OUT1: track 0.00 -> 28.6 mm
- net SHB: track 0.00 -> 26.8 mm, vias 0 -> 42
- net INHC: track 0.00 -> 26.7 mm, vias 0 -> 2
- net GLB: track 0.00 -> 26.6 mm, vias 0 -> 2
- net OUT2: track 0.00 -> 25.3 mm
- net +3V: track 0.00 -> 24.7 mm, vias 0 -> 2
- net INLA: track 0.00 -> 24.7 mm, vias 0 -> 2
- net INLB: track 0.00 -> 24.7 mm, vias 0 -> 2
- net INHA: track 0.00 -> 24.3 mm, vias 0 -> 2
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- added copper zone on B.Cu, net GND
- added copper zone on F.Cu, net GND
- added copper zone on In1.Cu, net GND
- added copper zone on In2.Cu, net GND
- added copper zone on B.Cu, net SHA
- added copper zone on F.Cu, net SHA
- added copper zone on In1.Cu, net SHA
- added copper zone on In2.Cu, net SHA
- added copper zone on B.Cu, net SHB
- added copper zone on F.Cu, net SHB
- added copper zone on In1.Cu, net SHB
- added copper zone on In2.Cu, net SHB
- added copper zone on B.Cu, net SHC
- added copper zone on F.Cu, net SHC
- added copper zone on In1.Cu, net SHC
- added copper zone on In2.Cu, net SHC
- added copper zone on In2.Cu, net VCC
- removed copper zone on F.Cu, net /FETs/HalfBridgeA/MP
- removed copper zone on F.Cu, net /FETs/HalfBridgeB/MP
- removed copper zone on F.Cu, net /FETs/HalfBridgeC/MP
