File: Hardware/KiCad_FOC-ESC/KiCad_FOC-ESC.kicad_pcb (KiCad board)
At the start: 6 copper layers, 51 x 46 mm, 74 parts, among them IC1 TCAN3414DDFR, IC2 TSC1801BILT, IC3 TSC1801BILT, IC4 TSC1801BILT, IC5 REF2030AIDDCR, IC6 MA702GQ-P, IC901 DRV8320SRTVR, J1 Conn_01x06, J2 Prog, J201 GSB1C41110SSHR, Q1 NTTFS5D6N08XLTAG, Q2 NTTFS5D6N08XLTAG, Q3 NTTFS5D6N08XLTAG, Q4 NTTFS5D6N08XLTAG, Q5 NTTFS5D6N08XLTAG, Q6 NTTFS5D6N08XLTAG, U1 STM32G473RCTx, U3 MT6701CT, U802 ZLDO1117Q, Y1 ASDDV-16.000MHZ-LR-T

Commit message: added:ferrite bead
Parts:
- added C23: 100nF, Capacitor_SMD:C_0402_1005Metric, F.Cu at (125.7, 78.4)
- added C24: 100nF, Capacitor_SMD:C_0402_1005Metric, F.Cu at (130.4, 83.7)
- added C25: 100nF, Capacitor_SMD:C_0402_1005Metric, F.Cu at (127.7, 80.2)
- added FB1: MPZ1608Y600BTA00, SamacSys_Parts:BEADC1608X95N, F.Cu at (127.7, 78.5)
- R7, R8: moved to B.Cu
- moved R7 65.6 mm to (125.8, 70.6)
- moved R8 64.6 mm to (123.8, 69.9)
- moved J201 33.4 mm to (126.2, 64.3)
- moved C6 6.06 mm to (130.0, 79.3), turned to 90 degrees
- moved C8 2.72 mm to (123.7, 79.4), turned to 0 degrees
- moved C9 1.05 mm to (123.7, 78.2)
- moved C1 0.40 mm to (130.6, 65.3)
- moved C16 0.40 mm to (138.0, 92.1)
- moved R2 0.40 mm to (137.5, 67.7)
- moved R3 0.40 mm to (137.5, 68.6)
- moved C901 0.40 mm to (142.2, 80.6)
- moved C902 0.40 mm to (134.4, 82.6)
- moved C903 0.40 mm to (134.4, 84.1)
- moved C904 0.40 mm to (135.9, 80.3)
- moved Q5 0.40 mm to (138.4, 100.6)
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Connections:
- C6 pad 1: +3V3 -> GND
- C6 pad 2: GND -> +3V3
- IC6 pad 13: unconnected-(IC6-VDD-Pad13) -> +3V3
- IC6 pad 17: unconnected-(IC6-GND_2-Pad17) -> GND
- IC6 pad 2: unconnected-(IC6-A-Pad2) -> A
- IC6 pad 3: unconnected-(IC6-Z-Pad3) -> Z
- IC6 pad 6: unconnected-(IC6-B-Pad6) -> B
- IC6 pad 8: unconnected-(IC6-GND_1-Pad8) -> GND
- U1 pad 29: +3V3 -> Net-(U1-VDDA)
- U3 pad 1: unconnected-(U3-VDD-Pad1) -> +3V3
- U3 pad 4: unconnected-(U3-GND-Pad4) -> GND
- U3 pad 6: unconnected-(U3-A-Pad6) -> A
- U3 pad 7: unconnected-(U3-B-Pad7) -> B
- U3 pad 8: unconnected-(U3-Z-Pad8) -> Z
Routing:
- net +5V: track 0.00 -> 19.0 mm
- net +3V3: track 181.3 -> 197.6 mm
- net GND: track 37.0 -> 42.9 mm, vias 122 -> 131
- net Z: track 0.00 -> 5.16 mm
- net B: track 0.00 -> 4.87 mm
- net +3V: track 24.3 -> 20.1 mm
- net Net-(U1-VDDA): track 0.00 -> 3.87 mm
- net Net-(J201-CC2): track 0.00 -> 3.80 mm
- net USB+: track 2.97 -> 5.50 mm
- net Net-(J201-CC1): track 0.00 -> 2.50 mm
- net USB-: track 2.97 -> 4.97 mm
- net CANRX: track 16.1 -> 17.8 mm
- net VCC: track 32.8 -> 34.4 mm
- net A: track 0.00 -> 1.53 mm
- net CANTX: track 16.7 -> 17.6 mm
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