File: Hardware/KiCad_FOC-ESC/Vref_1V65.kicad_sch (KiCad schematic)
At the start: 1 part, among them IC5 AZ431LBNTR-G1

Commit message: inited Software (#7)
Parts:
- IC5: footprint SOT96P240X105-3N -> SamacSys_Parts:SOT96P240X105-3N
Changed lines of the file:
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@@
 			)
 		)
-		(property "Footprint" "SOT96P240X105-3N"
+		(property "Footprint" "SamacSys_Parts:SOT96P240X105-3N"
 			(at 76.2 141.91 0)
 			(hide yes)

Commit message: Foc esc/comp manage (#8)
* inited Software

* ready
Parts:
- removed IC5: AZ431LBNTR-G1, SamacSys_Parts:SOT96P240X105-3N, symbol SamacSys_Parts:AZ431LBNTR-G1
- added PS1: REF3030AIDBZR, SamacSys_Parts:SOT96P240X105-3N, symbol SamacSys_Parts:REF3030AIDBZR
Changed lines of the file:
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@@
 	(paper "A4")
 	(symbol
-		(lib_id "SamacSys_Parts:AZ431LBNTR-G1")
-		(at 46.99 46.99 0)
+		(lib_id "SamacSys_Parts:REF3030AIDBZR")
+		(at 62.23 48.26 0)
 		(unit 1)
 		(body_style 1)
@@
 		(dnp no)
 		(fields_autoplaced yes)
-		(property "Reference" "IC5"
-			(at 63.5 39.37 0)
+		(property "Reference" "PS1"
+			(at 74.93 40.64 0)
 			(show_name no)
 			(do_not_autoplace no)
@@
 			)
 		)
-		(property "Value" "AZ431LBNTR-G1"
-			(at 63.5 41.91 0)
+		(property "Value" "REF3030AIDBZR"
+			(at 74.93 43.18 0)
 			(show_name no)
 			(do_not_autoplace no)
@@
 			)
 		)
-		(property "Datasheet" "https://www.diodes.com//assets/Datasheets/AZ431L.pdf"
-			(at 76.2 241.91 0)
+		(property "Datasheet" "http://www.ti.com/lit/gpn/ref3030"
+			(at 83.82 243.18 0)
 			(hide yes)
 			(show_name no)
@@
 			)
 		)
-		(property "Description" "Diodes Inc AZ431LBNTR-G1, Adjustable Shunt Adjustable Voltage Reference 1.24V, 1%, 3-Pin SOT-23"
-			(at 46.99 46.99 0)
+		(property "Description" "3.0V 50ppm/Degrees C, 50uA in SOT23-3 Series (Bandgap) Voltage Reference"
+			(at 62.23 48.26 0)
 			(hide yes)
 			(show_name no)
@@
 			)
 		)
-		(property "Height" "1.05"
-			(at 76.2 441.91 0)
+		(property "Height" "1.12"
+			(at 83.82 443.18 0)
 			(hide yes)
 			(show_name no)
@@
 			)
 		)
-		(property "Mouser Part Number" "621-AZ431LBNTR-G1"
-			(at 76.2 541.91 0)
+		(property "Mouser Part Number" "595-REF3030AIDBZR"
+			(at 83.82 543.18 0)
 			(hide yes)
 			(show_name no)
@@
 			)
 		)
-		(property "Mouser Price/Stock" "https://www.mouser.co.uk/ProductDetail/Diodes-Incorporated/AZ431LBNTR-G1?qs=eSfX1CQlHqpnB6E3RI3D7g%3D%3D"
-			(at 76.2 641.91 0)
+		(property "Mouser Price/Stock" "https://www.mouser.co.uk/ProductDetail/Texas-Instruments/REF3030AIDBZR?qs=sSOk4GDDv7zukMymvC3FQw%3D%3D"
+			(at 83.82 643.18 0)
 			(hide yes)
 			(show_name no)
@@
 			)
 		)
-		(property "Manufacturer_Name" "Diodes Incorporated"
-			(at 76.2 741.91 0)
+		(property "Manufacturer_Name" "Texas Instruments"
+			(at 83.82 743.18 0)
 			(hide yes)
 			(show_name no)
@@
 			)
 		)
-		(property "Manufacturer_Part_Number" "AZ431LBNTR-G1"
-			(at 76.2 841.91 0)
+		(property "Manufacturer_Part_Number" "REF3030AIDBZR"
+			(at 83.82 843.18 0)
 			(hide yes)
 			(show_name no)
@@
 			)
 		)
+		(pin "2"
+		)
 		(pin "1"
 		)
 		(pin "3"
 		)
-		(pin "2"
-		)
 		(instances
 			(project "KiCad_FOC-ESC"
 				(path "/5aa129d7-7a76-48d9-8008-691cf751c140/044506da-39ce-4369-ac96-5c2641096961"
-					(reference "IC5")
+					(reference "PS1")
 					(unit 1)
 				)

Commit message: initial connections
Parts:
- removed PS1: REF3030AIDBZR, SamacSys_Parts:SOT96P240X105-3N, symbol SamacSys_Parts:REF3030AIDBZR
- added C13, C17, C19: 100nF, Capacitor_SMD:C_0402_1005Metric, symbol Device:C
- added IC5: REF2030AIDDCR, SOT95P280X110-5N, symbol SamacSys_Parts:REF2030AIDDCR
Connections:
- new net +1V5: C17.2, IC5.1 (VBIAS)
- new net +3V: C19.2, IC5.5 (VREF)
- new net +5V: C13.2, IC5.3 (EN), IC5.4 (VIN)
- new net GND: C13.1, C17.1, C19.1, IC5.2 (GND)
