File: Hardware/KiCad_FOC-ESC/CAN.kicad_sch (KiCad schematic)
At the start: 5 parts, among them IC1 TCAN3414DDFR, J1 Conn_01x06

Commit message: Foc esc/stm32 idefo cinit (#22)
* edited FOC-ESC connections

* added CAN
Parts:
- added C22: 100nF, Capacitor_SMD:C_0402_1005Metric, symbol Device:C
- R2, R3: footprint Resistor_SMD:R_0603_1608Metric -> Resistor_SMD:R_0402_1005Metric
Connections:
- net +3V3: now also J1.1 (Pin_1), C22.1
- net GND: now also C22.2
- net CANH renamed CAN+
- net CANL renamed CAN-
