File: Hardware/KiCad_FOC-ESC/DRV8320S.kicad_sch (KiCad schematic)
At the start: 10 parts, among them IC901 DRV8320SRTVR

Commit message: Foc esc/stm32 idefo cinit (#22)
* edited FOC-ESC connections

* added CAN
Changed lines of the file:
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@@
+	)
+	(junction
+		(at 151.13 130.81)
+		(diameter 0)
+		(color 0 0 0 0)
 	)
 	(junction
@@
 		(color 0 0 0 0)
 	)
-	(junction
-		(at 151.13 130.81)
-		(diameter 0)
-		(color 0 0 0 0)
-	)
 	(wire
 		(pts
 			(xy 96.52 73.66) (xy 96.52 76.2)
+		)
+		(stroke
+			(width 0)
+			(type default)
+		)
+	)
+	(wire
+		(pts
+			(xy 151.13 135.89) (xy 151.13 130.81)
 		)
 		(stroke
@@
 	(symbol
 		(lib_id "power:GND")
-		(at 151.13 130.81 0)
+		(at 151.13 135.89 0)
 		(unit 1)
 		(body_style 1)
@@
 		(fields_autoplaced yes)
 		(property "Reference" "#PWR023"
-			(at 151.13 137.16 0)
+			(at 151.13 142.24 0)
 			(hide yes)
 			(show_name no)
@@
 		)
 		(property "Value" "GND"
+			(at 151.13 140.97 0)
+			(show_name no)
+			(do_not_autoplace no)
+			(effects
+				(font
+					(size 1.27 1.27)
+				)
+			)
+		)
+		(property "Footprint" ""
 			(at 151.13 135.89 0)
-			(show_name no)
-			(do_not_autoplace no)
-			(effects
-				(font
-					(size 1.27 1.27)
-				)
-			)
-		)
-		(property "Footprint" ""
-			(at 151.13 130.81 0)
 			(hide yes)
 			(show_name no)
@@
 		)
 		(property "Datasheet" ""
-			(at 151.13 130.81 0)
+			(at 151.13 135.89 0)
 			(hide yes)
 			(show_name no)
@@
 		)
 		(property "Description" "Power symbol creates a global label with name \"GND\" , ground"
-			(at 151.13 130.81 0)
-			(hide yes)
-			(show_name no)
+			(at 151.13 135.89 0)
+			(hide yes)
+			(show_name no)
